File: retro_gaming.kicad_pcb (KiCad board)
At the start: 2 copper layers, 11 parts, among them J1 alim, J2 USB-C, J3 DF40C, J4 DF40C, J5 1-84953-5, J6 Output Speaker, U1 BQ25895RTWR, U2 TS3USB221RSER, U3 MAX98357AETE_T

Commit message: PCB Started
Parts:
- added C1: 22uF, Capacitor_SMD:C_0805_2012Metric, F.Cu at (74.7, 160.6)
- added C10: 4.7uF, Capacitor_SMD:C_0805_2012Metric, F.Cu at (83.6, 163.6)
- added C11: 10uF, Capacitor_SMD:C_0805_2012Metric, F.Cu at (83.6, 166.6)
- added C12: 22uF, Capacitor_SMD:C_0805_2012Metric, F.Cu at (83.6, 169.6)
- added C13: 22uF, Capacitor_SMD:C_0805_2012Metric, F.Cu at (88.1, 160.6)
- added C14: 22uF, Capacitor_SMD:C_0805_2012Metric, F.Cu at (88.1, 163.6)
- added C15: 4.7uF, Capacitor_SMD:C_0805_2012Metric, F.Cu at (88.1, 166.6)
- added C16: 10nF, Capacitor_SMD:C_0805_2012Metric, F.Cu at (88.1, 169.6)
- added C2: 22uF, Capacitor_SMD:C_0805_2012Metric, F.Cu at (74.7, 163.6)
- added C3: 10uF, Capacitor_SMD:C_0805_2012Metric, F.Cu at (74.7, 166.6)
- added C4: 10uF, Capacitor_SMD:C_0805_2012Metric, F.Cu at (74.7, 169.6)
- added C5: 10nF, Capacitor_SMD:C_0805_2012Metric, F.Cu at (79.2, 160.6)
- added C6: 22uF, Capacitor_SMD:C_0805_2012Metric, F.Cu at (79.2, 163.6)
- added C7: 22uF, Capacitor_SMD:C_0805_2012Metric, F.Cu at (79.2, 166.6)
- added C8: 10uF, Capacitor_SMD:C_0805_2012Metric, F.Cu at (79.2, 169.6)
- added C9: 47nF, Capacitor_SMD:C_0805_2012Metric, F.Cu at (83.6, 160.6)
- added D1: 1N4148, Diode_THT:D_DO-35_SOD27_P7.62mm_Horizontal, F.Cu at (105.1, 167.7)
- added D2: 1N4148, Diode_THT:D_DO-35_SOD27_P7.62mm_Horizontal, F.Cu at (105.1, 171.2)
- added D3: LED, LED_SMD:LED_0805_2012Metric, F.Cu at (116.5, 167.4)
- added D4: LED, LED_SMD:LED_0805_2012Metric, F.Cu at (127.5, 158.3)
- added J10: Speaker, Connector_PinSocket_2.00mm:PinSocket_1x02_P2.00mm_Vertical, F.Cu at (115.2, 153.2)
- added J7: MDT420M01501, MDT420M01501:AMPHENOL_MDT420M01501, F.Cu at (137.0, 153.0)
- added J8: DM3D-SF, DM3D_SF:HRS_DM3D-SF, F.Cu at (157.7, 132.3)
- added J9: 1-84953-5, 1_84953_5:TE_1-84953-5, F.Cu at (137.5, 136.4)
- added L2: 2.2uH, Inductor_SMD:L_1008_2520Metric, F.Cu at (115.6, 125.6)
- added L3: 2.2uH, Inductor_SMD:L_1008_2520Metric, F.Cu at (115.6, 129.4)
- added R1: 5.1k, Resistor_SMD:R_0805_2012Metric, F.Cu at (165.5, 136.1)
- added R10: 30.1k, Resistor_SMD:R_0805_2012Metric, F.Cu at (96.9, 166.4)
- added R11: 5.23k, Resistor_SMD:R_0805_2012Metric, F.Cu at (96.9, 169.4)
- added R12: 260, Resistor_SMD:R_0805_2012Metric, F.Cu at (96.9, 172.3)
- added R13: 2.2K, Resistor_SMD:R_0805_2012Metric, F.Cu at (101.3, 160.5)
- added R14: 2.2K, Resistor_SMD:R_0805_2012Metric, F.Cu at (101.3, 163.5)
- added R15: 10k, Resistor_SMD:R_0805_2012Metric, F.Cu at (165.5, 142.0)
- added R16: 2.2K, Resistor_SMD:R_0805_2012Metric, F.Cu at (165.5, 144.9)
- added R17: 1M, Resistor_SMD:R_0603_1608Metric, F.Cu at (120.8, 167.2)
- added R18: 10k, Resistor_SMD:R_0805_2012Metric, F.Cu at (101.3, 166.4)
- added R19: 22k, Resistor_SMD:R_0805_2012Metric, F.Cu at (101.3, 169.4)
- added R2: 5.1k, Resistor_SMD:R_0805_2012Metric, F.Cu at (165.5, 139.0)
- added R3: 100k, Resistor_SMD:R_0805_2012Metric, F.Cu at (92.5, 160.5)
- added R4: 100k, Resistor_SMD:R_0805_2012Metric, F.Cu at (92.5, 163.5)
- added R5: 316k, Resistor_SMD:R_0805_2012Metric, F.Cu at (92.5, 166.4)
- added R6: 2.2K, Resistor_SMD:R_0805_2012Metric, F.Cu at (92.5, 169.4)
- added R7: 10k, Resistor_SMD:R_0805_2012Metric, F.Cu at (92.5, 172.3)
- added R8: 10k, Resistor_SMD:R_0805_2012Metric, F.Cu at (96.9, 160.5)
- added R9: 10k, Resistor_SMD:R_0805_2012Metric, F.Cu at (96.9, 163.5)
- added SW1: UP, Button_Switch_SMD:SW_Push_1P1T_NO_CK_KSC6xxG, F.Cu at (79.3, 123.9)
- added SW10: L2, Button_Switch_SMD:SW_Push_1P1T_NO_CK_KSC6xxG, F.Cu at (92.8, 155.1)
- added SW11: R1, Button_Switch_SMD:SW_Push_1P1T_NO_CK_KSC6xxG, F.Cu at (106.4, 123.9)
- added SW12: R2, Button_Switch_SMD:SW_Push_1P1T_NO_CK_KSC6xxG, F.Cu at (106.4, 131.7)
- added SW13: Start, Button_Switch_SMD:SW_Push_1P1T_NO_CK_KSC6xxG, F.Cu at (106.4, 139.5)
- added SW14: Select, Button_Switch_SMD:SW_Push_1P1T_NO_CK_KSC6xxG, F.Cu at (106.4, 147.3)
- added SW2: Left, Button_Switch_SMD:SW_Push_1P1T_NO_CK_KSC6xxG, F.Cu at (79.3, 131.7)
- added SW3: Right, Button_Switch_SMD:SW_Push_1P1T_NO_CK_KSC6xxG, F.Cu at (79.3, 139.5)
- added SW4: Down, Button_Switch_SMD:SW_Push_1P1T_NO_CK_KSC6xxG, F.Cu at (79.3, 147.3)
- added SW5: Y, Button_Switch_SMD:SW_Push_1P1T_NO_CK_KSC6xxG, F.Cu at (79.3, 155.1)
- added SW6: X, Button_Switch_SMD:SW_Push_1P1T_NO_CK_KSC6xxG, F.Cu at (92.8, 123.9)
- added SW7: B, Button_Switch_SMD:SW_Push_1P1T_NO_CK_KSC6xxG, F.Cu at (92.8, 131.7)
- added SW8: A, Button_Switch_SMD:SW_Push_1P1T_NO_CK_KSC6xxG, F.Cu at (92.8, 139.5)
- added SW9: L1, Button_Switch_SMD:SW_Push_1P1T_NO_CK_KSC6xxG, F.Cu at (92.8, 147.3)
- added TH1: 10k, Resistor_SMD:R_4020_10251Metric, F.Cu at (109.9, 162.5)
- added U4: TPS62823DLC, Package_SON:Texas_VSON-HR-8_1.5x2mm_P0.5mm, F.Cu at (120.0, 121.9)
- added U5: ADS1015IDGS, Package_SO:TSSOP-10_3x3mm_P0.5mm, F.Cu at (116.8, 142.6)
- added U6: MAX98357AETE_T, MAX98357AETE_T:QFN50P300X300X80-17N, F.Cu at (120.4, 153.8)
- J1: value alim -> UJ20-C-H-G-SMT-1-P16-TR; footprint Connector_PinSocket_2.54mm:PinSocket_1x02_P2.54mm_Vertical -> UJ20_C_H_G_SMT_1_P16_TR:SAMESKY_UJ20-C-H-G-SMT-1-P16-TR
- J2: value USB-C -> Conn_01x02_Socket; footprint UJ20_C_H_G_SMT_1_P16_TR:SAMESKY_UJ20-C-H-G-SMT-1-P16-TR -> Connector_PinSocket_2.00mm:PinSocket_1x02_P2.00mm_Vertical
- J5: value 1-84953-5 -> FFC3B11-05-T; footprint Conn_FPC_15p:TE_1-84953-5 -> FFC3B11:GCT_FFC3B11-05-T
- J6: value Output Speaker -> FFC3B11-05-T; footprint Connector_PinSocket_2.54mm:PinSocket_1x02_P2.54mm_Vertical -> FFC3B11:GCT_FFC3B11-05-T
- L1: value WE-PD_6050R -> 1uH; footprint 7447786002:WE-PD_6050R -> Inductor_SMD:L_1008_2520Metric
- U2: value TS3USB221RSER -> TPS61230ARNST; footprint TS3USB221RSER:RSE10 -> TPS61230A:IC_TPS61230ARNST
- U3: value MAX98357AETE_T -> TS3USB221RSER; footprint MAX98357AETE_T:QFN50P300X300X80-17N -> TS3USB221RSER:RSE10
- moved J4 76.4 mm to (138.0, 50.0)
- moved J2 62.4 mm to (165.3, 148.4)
- moved U3 53.8 mm to (116.1, 171.3)
- moved J5 48.7 mm to (156.5, 139.4)
- moved J3 39.2 mm to (138.0, 86.0)
- moved U1 36.7 mm to (116.8, 148.0)
- moved J6 30.7 mm to (156.5, 148.8)
- moved U2 29.0 mm to (119.9, 171.4)
- moved J1 28.1 mm to (138.0, 111.0)
- moved L1 17.1 mm to (115.6, 121.9)
- moved S1 11.3 mm to (118.2, 135.8)
Connections:
- net /INT renamed INT
- net /SDA renamed SDA
- J3 pad 24: unconnected-(J3-Pad24) -> GPIO26
- J3 pad 25: /DIN -> DIN
- J3 pad 26: /LRC -> LRC
- J3 pad 27: unconnected-(J3-Pad27) -> Power_keep
- J3 pad 28: unconnected-(J3-Pad28) -> GPIO13
- J3 pad 29: unconnected-(J3-Pad29) -> GPIO16
- J3 pad 30: unconnected-(J3-Pad30) -> GPIO6
- J3 pad 31: unconnected-(J3-Pad31) -> GPIO12
- J3 pad 34: unconnected-(J3-Pad34) -> GPIO5
- J3 pad 37: unconnected-(J3-Pad37) -> GPIO7
- J3 pad 38: unconnected-(J3-Pad38) -> GPIO11
- J3 pad 39: unconnected-(J3-Pad39) -> GPIO8
- J3 pad 40: unconnected-(J3-Pad40) -> GPIO9
- J3 pad 41: unconnected-(J3-Pad41) -> GPIO25
- J3 pad 44: unconnected-(J3-Pad44) -> GPIO10
- J3 pad 45: unconnected-(J3-Pad45) -> GPIO24
- J3 pad 46: unconnected-(J3-Pad46) -> GPIO22
- J3 pad 47: unconnected-(J3-Pad47) -> GPIO23
- J3 pad 48: unconnected-(J3-Pad48) -> GPIO27
- J3 pad 49: /BCLK -> BCLK
- J3 pad 50: unconnected-(J3-Pad50) -> GPIO17
- J3 pad 56: /CLK -> CLK
- J3 pad 57: unconnected-(J3-Pad57) -> SD_CLK
- J3 pad 61: unconnected-(J3-Pad61) -> SD_DAT3
- J3 pad 62: unconnected-(J3-Pad62) -> SD_CMD
- J3 pad 63: unconnected-(J3-Pad63) -> SD_DAT0
- J3 pad 67: unconnected-(J3-Pad67) -> SD_DAT1
- J3 pad 69: unconnected-(J3-Pad69) -> SD_DAT2
- J3 pad 80: /SCL0 -> SCL0
- J3 pad 82: /SDA0 -> SDA0
- J3 pad 84: 3V3 -> +3.3V
- J3 pad 86: 3V3 -> +3.3V
- J3 pad 88: 3V3 -> +3.3V
- J3 pad 90: 3V3 -> +3.3V
- J4 pad 10: unconnected-(J4-Pad10) -> REFCLK+
- J4 pad 12: unconnected-(J4-Pad12) -> REFCLK-
- J4 pad 16: unconnected-(J4-Pad16) -> PETp0
- J4 pad 18: unconnected-(J4-Pad18) -> PETn0
- J4 pad 22: unconnected-(J4-Pad22) -> PERp0
- J4 pad 24: unconnected-(J4-Pad24) -> PERn0
- J4 pad 3: /USB_N -> USB_N
- J4 pad 5: /USB_P -> USB_P
- J4 pad 75: /DSI1_DN0 -> DSI1_DN0
- J4 pad 77: /DSI1_DP0 -> DSI1_DP0
- J4 pad 81: /DSI1_DN1 -> DSI1_DN1
- J4 pad 83: /DSI1_DP1 -> DSI1_DP1
- J4 pad 87: /DSI1_CN -> DSI1_CN
- J4 pad 89: /DSI1_CP -> DSI1_CP
- J4 pad 9: unconnected-(J4-Pad9) -> PERST#
- J5 pad 1: GND -> +3.3V
- J5 pad 2: /DSI1_DN1 -> JG_AxeY
- J5 pad 3: /DSI1_DP1 -> JG_AxeX
- J5 pad 5: /DSI1_CN -> GPIO17
- J6 pad 1: Net-(J6-Pin_1) -> +3.3V
- J6 pad 2: Net-(J6-Pin_2) -> JD_AxeY
- L1 pad 1: Net-(U1-SW) -> V_SYS
- L1 pad 2: Net-(U1-SW__1) -> Net-(U2-SW)
- S1 pad 1: Net-(J1-Pin_2) -> V_SYS
- S1 pad 2: Net-(U1-OTG) -> Net-(D1-A)
- S1 pad 3: Net-(R7-Pad1) -> GND
- U1 pad 1: Net-(J2-VBUS) -> Vbus
- U1 pad 13: Net-(J1-Pin_2) -> Bat
- U1 pad 14: Net-(J1-Pin_2) -> Bat
- U1 pad 15: Net-(U1-SYS) -> V_SYS
- U1 pad 16: Net-(U1-SYS) -> V_SYS
- U1 pad 2: /CLK -> D_P
- U1 pad 20: Net-(U1-SW__1) -> Net-(U1-SW)
- U1 pad 22: Net-(U1-REGN) -> REGN
- U1 pad 23: +5V -> Net-(U1-PMID)
- U1 pad 24: /SEL -> DSEL
- U1 pad 25: unconnected-(U1-POWERPAD-Pad25) -> GND
- U1 pad 3: Net-(U1-D–) -> D_N
- U1 pad 5: /CLK -> CLK
- U1 pad 8: Net-(U1-OTG) -> GND
- U2 pad 1: /CLK -> Net-(U2-CBST)
- U2 pad 2: Net-(U1-D–) -> EN
- U2 pad 3: /USB_P -> Net-(U2-FB)
- U2 pad 4: /USB_N -> V_SYS
- U2 pad 5: GND -> Net-(U2-SW)
- U2 pad 7: Net-(J2-DN1) -> +5V
- U3 pad 1: /DIN -> D_P
- U3 pad 10: Net-(J6-Pin_1) -> +3.3V
- U3 pad 2: unconnected-(U3-GAIN_SLOT-Pad2) -> D_N
- U3 pad 3: GND -> USB_P
- U3 pad 4: Net-(U3-SD_MODE) -> USB_N
- U3 pad 5: (no net) -> GND
- U3 pad 6: (no net) -> GND
- U3 pad 7: +5V -> D-
- U3 pad 8: +5V -> D+
- U3 pad 9: Net-(J6-Pin_2) -> DSEL
